Commit message: feat: add colour

File: urdf/articulated_bot.xacro (robot description, xacro)
@@ -1,4 +1,5 @@
 <?xml version='1.0'?>
 <robot name="articulated_bot" xmlns:xacro="http://www.ros.org/wiki/xacro">
+  <xacro:include filename="$(find articulated_bot)/urdf/articulated_bot.gazebo" />
   <xacro:property name="wheel_length" value="0.05" />
   <xacro:property name="wheel_radius" value="0.1" />
@@ -37,5 +38,5 @@
       </geometry>
     </collision>
-    <visual name='chassis_visual'>
+    <visual>
       <origin xyz="-${chassis_x_offset} 0 0" rpy=" 0 0 0"/>
       <geometry>
@@ -43,5 +44,5 @@
       </geometry>
     </visual>
-    <visual name='back_chassis_link_visual'>
+    <visual>
       <origin xyz="-0.025 0 0" rpy=" 0 0 0"/>
       <geometry>
@@ -49,5 +50,5 @@
       </geometry>
     </visual>
-    <visual name='chassis_pin_visual'>
+    <visual>
       <origin xyz="0 0 0" rpy=" 0 0 0"/>
       <geometry>
@@ -71,5 +72,5 @@
       </geometry>
     </collision>
-    <visual name="left_wheel_visual">
+    <visual>
       <origin xyz="0 0 0" rpy=" 0 1.5707 1.5707"/>
       <geometry>
@@ -101,5 +102,5 @@
       </geometry>
     </collision>
-    <visual name="right_wheel_visual">
+    <visual>
       <origin xyz="0 0 0" rpy=" 0 1.5707 1.5707"/>
       <geometry>
@@ -140,5 +141,5 @@
       </geometry>
     </collision>
-    <visual name='chassis_visual'>
+    <visual>
       <origin xyz="${chassis_x_offset} 0 0" rpy=" 0 0 0"/>
       <geometry>
@@ -146,5 +147,5 @@
       </geometry>
     </visual>
-    <visual name='front_chassis_link_visual'>
+    <visual>
       <origin xyz="0.025 0 0" rpy=" 0 0 0"/>
       <geometry>
@@ -168,5 +169,5 @@
       </geometry>
     </collision>
-    <visual name="visual">
+    <visual>
       <origin xyz="0 0 0" rpy=" 0 1.5707 1.5707"/>
       <geometry>
@@ -198,5 +199,5 @@
       </geometry>
     </collision>
-    <visual name="visual">
+    <visual>
       <origin xyz="0 0 0" rpy=" 0 1.5707 1.5707"/>
       <geometry>
@@ -229,5 +230,5 @@
       </geometry>
     </collision>
-    <visual name='camera_visual'>
+    <visual>
       <origin xyz="0 0 0" rpy=" 0 0 0"/>
       <geometry>
@@ -260,5 +261,5 @@
       </geometry>
     </collision>
-    <visual name='hokuyo_visual'>
+    <visual>
       <origin xyz="0 0 0" rpy=" 0 0 0"/>
       <geometry>
